Commit message: feat(jackal_description): setup jackal_description for Miss configuration

File: jackal_description/urdf/accessories.urdf.xacro (robot description, xacro)
@@ -1,29 +1,9 @@
 <?xml version="1.0"?>
 <robot xmlns:xacro="http://www.ros.org/wiki/xacro">
-  <!--
-    As you add to this URDF, please be aware that both the robot and
-    simulation include it. You must retain compatibility with all of
-    the following launch files:
-    jackal_viz/launch/view_model.launch
-    jackal_gazebo/launch/jackal_world.launch
-    jackal_base/launch/base.launch
-  -->
-  <!-- Macros to generate standoffs for offset payload mounting. -->
   <xacro:include filename="$(find jackal_description)/urdf/accessories/standoffs.urdf.xacro" />
-  <!-- This optional plate mounts both the upgraded GPS and the Velodyne 3D LIDAR. -->
   <xacro:include filename="$(find jackal_description)/urdf/accessories/bridge_plate.urdf.xacro" />
-  <!-- 2D Lidars -->
-  <!-- <xacro:include filename="$(find lms1xx)/urdf/sick_lms1xx.urdf.xacro" />
-  <xacro:include filename="$(find jackal_description)/urdf/accessories/sick_lms1xx_mount.urdf.xacro" />-->
   <xacro:include filename="$(find jackal_description)/urdf/accessories/hokuyo_ust10.urdf.xacro" />
   <xacro:include filename="$(find jackal_description)/urdf/accessories/vlp16_mount.urdf.xacro" />
   <xacro:include filename="$(find jackal_description)/urdf/accessories/hdl32_mount.urdf.xacro" />
-  <!--
-    Add primary/secondary 2D lidar sensors.  By default these are SICK LMS1xx but can be changed with the
-    JACKAL_LASER_MODEL and JACKAL_LASER_SECONDARY_MODEL environment variables. Valid model designations are:
-    - lms1xx (default) :: SICK LMS1xx
-    - ust10            :: Hokuyo UST10
-  -->
-  <!-- Primary 2D Lidar -->
   <xacro:if value="$(optenv JACKAL_LASER 0)">
     <xacro:property name="mount" value="$(optenv JACKAL_LASER_MOUNT front)" />
@@ -33,7 +13,5 @@
     <xacro:property name="parent" value="$(optenv JACKAL_LASER_PARENT ${mount}_mount)" />
     <xacro:property name="lidar_model" value="$(optenv JACKAL_LASER_MODEL ust10)" />
-    <!-- SICK LMS1xx -->
     <xacro:if value="${lidar_model == 'lms1xx'}">
-      <!-- Mount Enabled -->
       <xacro:if value="${tower}">
         <xacro:sick_lms1xx_mount topic="${topic}" prefix="${prefix}" parent_link="${parent}">
@@ -41,5 +19,4 @@
         </xacro:sick_lms1xx_mount>
       </xacro:if>
-      <!-- Mount Disabled -->
       <xacro:unless value="${tower}">
         <xacro:sick_lms1xx frame="${prefix}_laser" topic="${topic}" />
@@ -57,5 +34,4 @@
       </xacro:unless>
     </xacro:if>
-    <!-- Hokuyo UST10 -->
     <xacro:if value="${lidar_model == 'ust10'}">
       <xacro:hokuyo_ust10_mount topic="${topic}" prefix="${prefix}" parent_link="${parent}">
@@ -64,5 +40,4 @@
     </xacro:if>
   </xacro:if>
-  <!-- Secondary 2D Lidar -->
   <xacro:if value="$(optenv JACKAL_LASER_SECONDARY 0)">
     <xacro:property name="mount" value="$(optenv JACKAL_LASER_SECONDARY_MOUNT rear)" />
@@ -72,7 +47,5 @@
     <xacro:property name="parent" value="$(optenv JACKAL_LASER_SECONDARY_PARENT ${mount}_mount)" />
     <xacro:property name="lidar_model" value="$(optenv JACKAL_LASER_SECONDARY_MODEL ust10)" />
-    <!-- SICK LMS1xx -->
     <xacro:if value="${lidar_model == 'lms1xx'}">
-      <!-- Mount Enabled -->
       <xacro:if value="${tower}">
         <xacro:sick_lms1xx_mount topic="${topic}" prefix="${prefix}" parent_link="${parent}">
@@ -80,5 +53,4 @@
         </xacro:sick_lms1xx_mount>
       </xacro:if>
-      <!-- Mount Disabled -->
       <xacro:unless value="${tower}">
         <xacro:sick_lms1xx frame="${prefix}_laser" topic="${topic}" />
@@ -96,5 +68,4 @@
       </xacro:unless>
     </xacro:if>
-    <!-- Hokuyo UST10 -->
     <xacro:if value="${lidar_model == 'ust10'}">
       <xacro:hokuyo_ust10_mount topic="${topic}" prefix="${prefix}" parent_link="${parent}">
@@ -103,10 +74,4 @@
     </xacro:if>
   </xacro:if>
-  <!--
-    Add a 3D lidar sensor.  By default this is a Velodyne VLP16 but can be changed with the
-    JACKAL_LASER_3D_MODEL environment variable. Valid model designations are:
-    - vlp16 (default)  :: Velodyne VLP16
-    - vlp32e           :: Velodyne HDL-32E
-  -->
   <xacro:if value="$(optenv JACKAL_LASER_3D 0)">
     <xacro:property name="mount" value="$(optenv JACKAL_LASER_3D_MOUNT mid)" />
@@ -116,5 +81,4 @@
     <xacro:property name="parent" value="$(optenv JACKAL_LASER_3D_PARENT ${mount}_mount)" />
     <xacro:property name="lidar_3d_model" value="$(optenv JACKAL_LASER_3D_MODEL vlp16)" />
-    <!-- Velodyne VLP16 -->
     <xacro:if value="${lidar_3d_model == 'vlp16'}">
       <xacro:vlp16_mount topic="${topic}" tower="${tower}" prefix="${prefix}" parent_link="${parent}" >
@@ -122,5 +86,4 @@
       </xacro:vlp16_mount>
     </xacro:if>
-    <!-- Velodyne HDL-32E -->
     <xacro:if value="${lidar_3d_model == 'hdl32e'}">
       <xacro:hdl32e_mount topic="${topic}" tower="${tower}" prefix="${prefix}" parent_link="${parent}" >
@@ -129,10 +92,4 @@
     </xacro:if>
   </xacro:if>
-  <!--
-    Add a Nav. Sat. By default this is a Novatel Smart6, but can be changed with the
-    JACKAL_NAVSAT_MODEL environment variable. Valid model designations are:
-    - smart6 (default)    :: Novatel Smart6
-    - smart7              :: Novatel Smart7
-  -->
   <xacro:include filename="$(find jackal_description)/urdf/accessories/novatel_smart6.urdf.xacro" />
   <xacro:include filename="$(find jackal_description)/urdf/accessories/novatel_smart7.urdf.xacro" />
@@ -143,8 +100,6 @@
     <xacro:property name="parent" value="$(optenv JACKAL_NAVSAT_PARENT ${mount}_mount)" />
     <xacro:property name="navsat_model" value="$(optenv JACKAL_NAVSAT_MODEL smart6)" />
-    <!--- Novotel Smart6 -->
     <xacro:if value="${navsat_model == 'smart6'}">
       <xacro:novatel_smart6 prefix="${prefix}"/>
-      <!-- Tower Enabled -->
       <xacro:if value="${tower}">
         <xacro:bridge_plate prefix="${prefix}" parent="${parent}" height="$(optenv JACKAL_NAVSAT_HEIGHT 0.1)">
@@ -157,5 +112,4 @@
         </joint>
       </xacro:if>
-      <!-- Tower Disabled -->
       <xacro:unless value="${tower}">
         <joint name="${prefix}_navsat_joint" type="fixed">
@@ -166,8 +120,6 @@
       </xacro:unless>
     </xacro:if>
-    <!-- Novotel Smart7 -->
     <xacro:if value="${navsat_model == 'smart7'}">
       <xacro:novatel_smart7 prefix="${prefix}"/>
-      <!-- Tower Enabled -->
       <xacro:if value="${tower}">
         <xacro:novatel_smart7_stand prefix="${prefix}" parent="${parent}" height="$(optenv JACKAL_NAVSAT_HEIGHT 0.145)">
@@ -180,5 +132,4 @@
         </joint>
       </xacro:if>
-      <!-- Tower Disabled -->
       <xacro:unless value="${tower}">
         <joint name="${prefix}_navsat_joint" type="fixed">
@@ -190,14 +141,5 @@
     </xacro:if>
   </xacro:if>
-  <!--
-    Add Cameras.
-    - JACKAL_FLEA3
-    - JACKAL_STEREO_FLEA3
-    - JACKAL_BB2
-  -->
-  <!-- Common camera mounts and accessory URDFs. -->
   <xacro:include filename="$(find jackal_description)/urdf/accessories/camera_mount.urdf.xacro" />
-  <!--xacro:include filename="$(find pointgrey_camera_description)/urdf/pointgrey_flea3.urdf.xacro" /-->
-  <!-- If enabled, generate the flea3 camera payload with a tilt of 30 degrees. -->
   <xacro:if value="$(optenv JACKAL_FLEA3 0)">
     <xacro:property name="name" value="$(optenv JACKAL_FLEA3_NAME front)" />
@@ -210,5 +152,4 @@
       camera_x="0.0754" camera_y="0.029" camera_z="0.029"
       camera_mass="0.085" hfov="1.0471975512" fps="60" width="640" height="512"/>
-    <!-- Mount Enabled -->
     <xacro:if value="${tower}">
       <xacro:camera_mount prefix="${prefix}" tilt="${tilt}"/>
@@ -225,5 +166,4 @@
       </joint>
     </xacro:if>
-    <!-- Mount Disabled -->
     <xacro:unless value="${tower}">
       <link name="${prefix}_camera_base"/>
@@ -243,6 +183,4 @@
   </xacro:if>
   <xacro:include filename="$(find jackal_description)/urdf/accessories/stereo_camera_mount.urdf.xacro" />
-  <!-- If enabled, generates a pair of flea3 cameras for stereo vision with a tilt of 30 degrees. -->
-  <!-- Disabled temporarily due to metapackage issue. -->
   <xacro:if value="$(optenv JACKAL_STEREO_FLEA3 0)">
     <xacro:property name="tilt" value="$(optenv JACKAL_FLEA3_TILT 0.5236)"/>
@@ -277,8 +215,4 @@
     </joint>
   </xacro:if>
-  <!-- If enabled, generate the bumblebee2 camera payload with a tilt of 0 degrees. -->
-  <!--xacro:include filename="$(find pointgrey_camera_description)/urdf/pointgrey_bumblebee2.urdf.xacro" /-->
-  <!-- If enabled, generate the bumblebee2 camera payload with a tilt of 0 degrees. -->
-  <!-- Disabled temporarily due to metapackage issue. -->
   <xacro:if value="$(optenv JACKAL_BB2 0)">
     <xacro:property name="tilt" value="$(optenv JACKAL_BB2_TILT 0)" />
@@ -289,5 +223,4 @@
     <xacro:property name="parent" value="$(optenv JACKAL_BB2_PARENT ${mount}_mount)"/>
     <xacro:BB2-08S2C-38 frame="${prefix}_camera" name="${name}" />
-    <!-- Mount Enabled -->
     <xacro:if value="${tower}">
       <xacro:camera_mount prefix="${prefix}" tilt="${tilt}"/>
@@ -304,5 +237,4 @@
       </joint>
     </xacro:if>
-    <!-- Mount Disabled -->
     <xacro:unless value="${tower}">
       <link name="${prefix}_camera_base" type="fixed"/>
@@ -320,5 +252,4 @@
     </xacro:unless>
   </xacro:if>
-  <!-- Fender Accessories -->
   <xacro:if value="$(optenv JACKAL_FRONT_ACCESSORY_FENDER 0)">
     <xacro:include filename="$(find jackal_description)/urdf/accessories/hokuyo_ust10.urdf.xacro" />

File: jackal_description/urdf/accessories/vlp16_mount.urdf.xacro (robot description, xacro)
@@ -1,92 +1,99 @@
 <robot xmlns:xacro="http://wiki.ros.org/xacro">
   <xacro:include filename="$(find velodyne_description)/urdf/VLP-16.urdf.xacro" />
-  <xacro:macro name="vlp16_mount" params="prefix parent_link topic height:=0.1 *origin">
-    <link name="${prefix}_vlp16_mount" />
-    <link name="${prefix}_vlp16_plate">
-      <visual>
-        <geometry>
-          <box size="0.1 0.1 0.002" />
-        </geometry>
-        <material name="black" />
-        <origin xyz="0 0 -0.001" rpy="0 0 0" />
-      </visual>
-    </link>
-    <link name="${prefix}_vlp16_leg1">
-      <visual>
-        <geometry>
-          <cylinder length="${height}" radius="0.003" />
-        </geometry>
-        <material name="white">
-          <color rgba="1 1 1 1" />
-        </material>
-        <origin xyz="0 0 ${height/2}" rpy="0 0 0" />
-      </visual>
-    </link>
-    <link name="${prefix}_vlp16_leg2">
-      <visual>
-        <geometry>
-          <cylinder length="${height}" radius="0.003" />
-        </geometry>
-        <material name="white">
-          <color rgba="1 1 1 1" />
-        </material>
-        <origin xyz="0 0 ${height/2}" rpy="0 0 0" />
-      </visual>
-    </link>
-    <link name="${prefix}_vlp16_leg3">
-      <visual>
-        <geometry>
-          <cylinder length="${height}" radius="0.003" />
-        </geometry>
-        <material name="white">
-          <color rgba="1 1 1 1" />
-        </material>
-        <origin xyz="0 0 ${height/2}" rpy="0 0 0" />
-      </visual>
-    </link>
-    <link name="${prefix}_vlp16_leg4">
-      <visual>
-        <geometry>
-          <cylinder length="${height}" radius="0.003" />
-        </geometry>
-        <material name="white">
-          <color rgba="1 1 1 1" />
-        </material>
-        <origin xyz="0 0 ${height/2}" rpy="0 0 0" />
-      </visual>
-    </link>
-    <joint name="${prefix}_vlp16_mount_joint" type="fixed">
-      <parent link="${parent_link}" />
-      <child link="${prefix}_vlp16_mount" />
-      <xacro:insert_block name="origin" />
-    </joint>
-    <joint name="${prefix}_vlp16_leg1_joint" type="fixed">
-      <parent link="${prefix}_mount" />
-      <child link="${prefix}_vlp16_leg1" />
-      <origin xyz="0.05 0.05 0" rpy="0 0 0" />
-    </joint>
-    <joint name="${prefix}_vlp16_leg2_joint" type="fixed">
-      <parent link="${prefix}_mount" />
-      <child link="${prefix}_vlp16_leg2" />
-      <origin xyz="0.05 -0.05 0" rpy="0 0 0" />
-    </joint>
-    <joint name="${prefix}_vlp16_leg3_joint" type="fixed">
-      <parent link="${prefix}_mount" />
-      <child link="${prefix}_vlp16_leg3" />
-      <origin xyz="-0.05 0.05 0" rpy="0 0 0" />
-    </joint>
-    <joint name="${prefix}_vlp16_leg4_joint" type="fixed">
-      <parent link="${prefix}_mount" />
-      <child link="${prefix}_vlp16_leg4" />
-      <origin xyz="-0.05 -0.05 0" rpy="0 0 0" />
-    </joint>
-    <joint name="${prefix}_vlp16_plate_joint" type="fixed">
-      <parent link="${prefix}_vlp16_mount" />
-      <child link="${prefix}_vlp16_plate" />
-      <origin xyz="0 0 ${height}" rpy="0 0 0" />
-    </joint>
-    <xacro:VLP-16 parent="${prefix}_vlp16_plate" topic="${topic}">
-      <origin xyz="0 0 0" rpy="0 0 0" />
-    </xacro:VLP-16>
+  <xacro:macro name="vlp16_mount" params="prefix parent_link topic tower height:=0.1 *origin">
+    <xacro:if value="${tower}">
+      <link name="${prefix}_vlp16_mount" />
+      <link name="${prefix}_vlp16_plate">
+        <visual>
+          <geometry>
+            <box size="0.1 0.1 0.002" />
+          </geometry>
+          <material name="black" />
+          <origin xyz="0 0 -0.001" rpy="0 0 0" />
+        </visual>
+      </link>
+      <link name="${prefix}_vlp16_leg1">
+        <visual>
+          <geometry>
+            <cylinder length="${height}" radius="0.003" />
+          </geometry>
+          <material name="white">
+            <color rgba="1 1 1 1" />
+          </material>
+          <origin xyz="0 0 ${height/2}" rpy="0 0 0" />
+        </visual>
+      </link>
+      <link name="${prefix}_vlp16_leg2">
+        <visual>
+          <geometry>
+            <cylinder length="${height}" radius="0.003" />
+          </geometry>
+          <material name="white">
+            <color rgba="1 1 1 1" />
+          </material>
+          <origin xyz="0 0 ${height/2}" rpy="0 0 0" />
+        </visual>
+      </link>
+      <link name="${prefix}_vlp16_leg3">
+        <visual>
+          <geometry>
+            <cylinder length="${height}" radius="0.003" />
+          </geometry>
+          <material name="white">
+            <color rgba="1 1 1 1" />
+          </material>
+          <origin xyz="0 0 ${height/2}" rpy="0 0 0" />
+        </visual>
+      </link>
+      <link name="${prefix}_vlp16_leg4">
+        <visual>
+          <geometry>
+            <cylinder length="${height}" radius="0.003" />
+          </geometry>
+          <material name="white">
+            <color rgba="1 1 1 1" />
+          </material>
+          <origin xyz="0 0 ${height/2}" rpy="0 0 0" />
+        </visual>
+      </link>
+      <joint name="${prefix}_vlp16_mount_joint" type="fixed">
+        <parent link="${parent_link}" />
+        <child link="${prefix}_vlp16_mount" />
+        <xacro:insert_block name="origin" />
+      </joint>
+      <joint name="${prefix}_vlp16_leg1_joint" type="fixed">
+        <parent link="${prefix}_vlp16_mount" />
+        <child link="${prefix}_vlp16_leg1" />
+        <origin xyz="0.05 0.05 0" rpy="0 0 0" />
+      </joint>
+      <joint name="${prefix}_vlp16_leg2_joint" type="fixed">
+        <parent link="${prefix}_vlp16_mount" />
+        <child link="${prefix}_vlp16_leg2" />
+        <origin xyz="0.05 -0.05 0" rpy="0 0 0" />
+      </joint>
+      <joint name="${prefix}_vlp16_leg3_joint" type="fixed">
+        <parent link="${prefix}_vlp16_mount" />
+        <child link="${prefix}_vlp16_leg3" />
+        <origin xyz="-0.05 0.05 0" rpy="0 0 0" />
+      </joint>
+      <joint name="${prefix}_vlp16_leg4_joint" type="fixed">
+        <parent link="${prefix}_vlp16_mount" />
+        <child link="${prefix}_vlp16_leg4" />
+        <origin xyz="-0.05 -0.05 0" rpy="0 0 0" />
+      </joint>
+      <joint name="${prefix}_vlp16_plate_joint" type="fixed">
+        <parent link="${prefix}_vlp16_mount" />
+        <child link="${prefix}_vlp16_plate" />
+        <origin xyz="0 0 ${height}" rpy="0 0 0" />
+      </joint>
+      <xacro:VLP-16 parent="${prefix}_vlp16_plate" topic="${topic}">
+        <origin xyz="0 0 0" rpy="0 0 0" />
+      </xacro:VLP-16>
+    </xacro:if>
+    <xacro:unless value="${tower}">
+      <xacro:VLP-16 parent="${parent_link}" topic="${topic}">
+        <xacro:insert_block name="origin" />
+      </xacro:VLP-16>
+    </xacro:unless>
   </xacro:macro>
 </robot>

File: jackal_description/urdf/jackal.urdf.xacro (robot description, xacro)
@@ -59,6 +59,4 @@
       <axis xyz="0 1 0" />
     </joint>
-    <!-- In reality, Jackal has only two motors, one per side. However, it's more
-         straightforward for Gazebo to simulate as if there's an actuator per wheel. -->
     <transmission name="${prefix}_wheel_trans">
       <type>transmission_interface/SimpleTransmission</type>
@@ -104,13 +102,11 @@
     </collision>
     <inertial>
-      <!-- Center of mass -->
       <origin xyz="0.012  0.002 0.067" rpy="0 0 0"/>
       <mass value="16.523"/>
-      <!-- Moments of inertia: ( chassis without wheels ) -->
       <inertia
         ixx="0.3136" ixy="-0.0008" ixz="0.0164"
         iyy="0.3922" iyz="-0.0009"
         izz="0.4485"/>
-      </inertial>
+    </inertial>
   </link>
   <xacro:unless value="$(optenv JACKAL_FRONT_ACCESSORY_FENDER 0)">
@@ -176,8 +172,4 @@
     <child link="rear_fender_link" />
   </joint>
-  <!-- TODO: Make this internal_imu_link or something, and use a mixed-in xacro
-       to supply the joint between it and imu_link. This is important so that imu_link
-       always points to the "active" IMU. When an upgrade IMU is connected, the
-       internal_imu_link should remain, but imu_link should point to the upgrade one. -->
   <link name="imu_link">
     <inertial>
@@ -191,5 +183,4 @@
     <child link="imu_link" />
   </joint>
-  <!-- TODO: Same note as applies to imu_link -->
   <link name="navsat_link">
     <visual>
@@ -224,5 +215,4 @@
     <origin xyz="${mount_spacing} 0 0" />
   </joint>
-  <!-- ROS2 controls -->
   <ros2_control name="jackal_hardware" type="system">
     <hardware>
@@ -256,13 +246,7 @@
     </joint>
   </ros2_control>
-  <!-- Bring in simulation data for Gazebo. -->
   <xacro:if value="$(arg is_sim)">
     <xacro:include filename="$(find jackal_description)/urdf/jackal.gazebo" />
   </xacro:if>
-  <!-- Optional standard accessories, including their simulation data. The rendering
-       of these into the final description is controlled by optenv variables, which
-       default each one to off.-->
-  <xacro:include filename="$(find jackal_description)/urdf/accessories.urdf.xacro" />
-  <!-- Optional custom includes. -->
-  <xacro:include filename="$(optenv JACKAL_URDF_EXTRAS empty.urdf)" />
+  <xacro:include filename="$(find jackal_description)/urdf/miss_sensors.urdf.xacro" />
 </robot>
