Commit message: refactor(jackal_description): move 3d lidar position and update its references to faster loading

File: jackal_description/urdf/miss_sensors.urdf.xacro (robot description, xacro)
@@ -2,6 +2,6 @@
   <xacro:include filename="$(find jackal_description)/urdf/accessories/hokuyo_ust10.urdf.xacro" />
   <xacro:include filename="$(find jackal_description)/urdf/accessories/_d435.urdf.xacro" />
-  <xacro:include filename="$(find velodyne_description)/urdf/VLP-16.urdf.xacro" />
-  <xacro:hokuyo_ust10_mount topic="/front/scan" prefix="front" parent_link="front_mount">
+  <xacro:include filename="$(find jackal_description)/urdf/accessories/_vlp16.urdf.xacro" />
+  <xacro:hokuyo_ust10_mount topic="/rear/scan" prefix="rear" parent_link="rear_mount">
     <origin xyz="0 0 0" rpy="0 0 0" />
   </xacro:hokuyo_ust10_mount>
@@ -10,5 +10,5 @@
     </xacro:sensor_d435>
   <xacro:VLP-16 parent="mid_mount">
-    <origin xyz="0 0 0" rpy="0 0 0" />
+    <origin xyz="0 0 0.76" rpy="0 0 0" />
   </xacro:VLP-16>
 </robot>
