Commit message: refactor: add misskal namespaces and prefix

File: jackal_description/urdf/jackal.urdf.xacro (robot description, xacro)
@@ -2,5 +2,5 @@
 <robot name="jackal" xmlns:xacro="http://www.ros.org/wiki/xacro">
   <xacro:arg name="is_sim" default="false" />
-  <xacro:arg name="prefix" default="" />
+  <xacro:arg name="prefix" default="misskal" />
   <xacro:arg name="gazebo_controllers" default="$(find jackal_control)/config/control.yaml" />
   <xacro:property name="PI" value="3.1415926535897931" />

File: jackal_description/urdf/miss_sensors.urdf.xacro (robot description, xacro)
@@ -10,5 +10,5 @@
     </xacro:sensor_d435>
   <xacro:VLP-16 parent="mid_mount">
-    <origin xyz="0 0 0.76" rpy="0 0 0" />
+    <origin xyz="0 0 0.69" rpy="0 0 0" />
   </xacro:VLP-16>
 </robot>

Commit message: feat(misskal_manipulator): add vx300s setup files

File: jackal_description/urdf/jackal.urdf.xacro (robot description, xacro)
@@ -215,4 +215,10 @@
     <origin xyz="${mount_spacing} 0 0" />
   </joint>
+<!-- $(arg robot_name)/$(arg base_link_frame) -->
+  <joint name="vx300s_joint" type="fixed">
+    <parent link="front_mount" />
+    <child link="misskal/vx300s_base" />
+    <origin xyz="${mount_spacing} 0 0.6" rpy="0 -${PI/2} ${PI}"/>
+  </joint>
   <ros2_control name="jackal_hardware" type="system">
     <hardware>

File: jackal_description/urdf/miss_sensors.urdf.xacro (robot description, xacro)
@@ -3,4 +3,5 @@
   <xacro:include filename="$(find jackal_description)/urdf/accessories/_d435.urdf.xacro" />
   <xacro:include filename="$(find jackal_description)/urdf/accessories/_vlp16.urdf.xacro" />
+  <xacro:include filename="$(find interbotix_xsarm_descriptions)/urdf/vx300s.urdf.xacro" />
   <xacro:hokuyo_ust10_mount topic="/rear/scan" prefix="rear" parent_link="rear_mount">
     <origin xyz="0 0 0" rpy="0 0 0" />
